File: BottleBlink.sch (KiCad schematic (older format))
At the start: 61 parts, among them J1 Arduino_Nano_v2.x, J2 Conn_01x06_Male, U1 LM2904

Commit message: Add changes based on review comments
Parts:
- added JP1: NM, Resistor_SMD:R_0603_1608Metric_Pad0.98x0.95mm_HandSolder, symbol Device:Jumper
- added JP2: Jumper, Resistor_SMD:R_0603_1608Metric_Pad0.98x0.95mm_HandSolder, symbol Device:Jumper
- added R1, R6: 10k, Resistor_SMD:R_0603_1608Metric_Pad0.98x0.95mm_HandSolder, symbol Device:R
- added SW1, SW2: SW_DPST_x2, Button_Switch_SMD:SW_SPST_EVQP0, symbol Switch:SW_DPST_x2
- renumbered JP1 to JP3, JP2 to JP4, JP3 to JP5, R8 to R10, R9 to R11, R10 to R12, R11 to R13, R1 to R2, R2 to R3, R3 to R4, R4 to R5, R5 to R7, R6 to R8, R7 to R9
Connections:
- net +3V3: now also JP2.2
- net +5VL: now also JP1.2
- net GND: now also SW1.1 (A), SW2.1 (A)
- net Btn1: now reaches J1.14 (D11)
- net Btn1: now also R1.2, SW1.2 (B)
- net Btn2: now reaches J1.15 (D12)
- net Btn2: now also R6.2, SW2.2 (B)
- new net: JP1.1, JP2.1, R1.1, R6.1

Commit message: Add LCSC numbers and QR code to PCB
Parts:
- C1: LCSC (none) -> C14663
- C10, C11, C12, C3, C4, C5, C6, C7, C8, C9: LCSC (none) -> C15849
- C13, C2: LCSC (none) -> C57112
- D30, D31: LCSC (none) -> C64898
- JP2, JP3, JP4, JP5: LCSC (none) -> C21189
- R1, R11, R13, R6: LCSC (none) -> C25804
- R10, R2: LCSC (none) -> C22961
- R12, R4, R7: LCSC (none) -> C21190
- R3, R8: LCSC (none) -> C4177
- R5: LCSC (none) -> C17477
- R9: LCSC (none) -> C23345
- U1: LCSC (none) -> C18229
Changed lines of the file:
@@
 F 2 "Resistor_SMD:R_0603_1608Metric_Pad0.98x0.95mm_HandSolder" H 4450 6800 50  0001 C CNN
 F 3 "~" H 4450 6800 50  0001 C CNN
+F 4 "C21189" H 4450 6800 50  0001 C CNN "LCSC"
 	1    4450 6800
 	1    0    0    -1
@@
 F 2 "Resistor_SMD:R_0603_1608Metric_Pad0.98x0.95mm_HandSolder" V 9430 5250 50  0001 C CNN
 F 3 "~" H 9500 5250 50  0001 C CNN
+F 4 "C23345" H 9500 5250 50  0001 C CNN "LCSC"
 	1    9500 5250
 	0    1    1    0
@@
 F 2 "Resistor_SMD:R_0805_2012Metric_Pad1.20x1.40mm_HandSolder" V 2030 4900 50  0001 C CNN
 F 3 "~" H 2100 4900 50  0001 C CNN
+F 4 "C17477" H 2100 4900 50  0001 C CNN "LCSC"
 	1    2100 4900
 	-1   0    0    1
@@
 F 2 "Resistor_SMD:R_0603_1608Metric_Pad0.98x0.95mm_HandSolder" V 680 6550 50  0001 C CNN
 F 3 "~" H 750 6550 50  0001 C CNN
+F 4 "C25804" H 750 6550 50  0001 C CNN "LCSC"
 	1    750  6550
 	1    0    0    -1
@@
 F 2 "Resistor_SMD:R_0603_1608Metric_Pad0.98x0.95mm_HandSolder" V 680 6900 50  0001 C CNN
 F 3 "~" H 750 6900 50  0001 C CNN
+F 4 "C25804" H 750 6900 50  0001 C CNN "LCSC"
 	1    750  6900
 	1    0    0    -1
@@
 F 2 "Package_SO:SOIC-8_3.9x4.9mm_P1.27mm" H 1350 6800 50  0001 C CNN
 F 3 "http://www.ti.com/lit/ds/symlink/lm358.pdf" H 1350 6800 50  0001 C CNN
+F 4 "C18229" H 1350 6800 50  0001 C CNN "LCSC"
 	2    1350 6800
 	1    0    0    -1
@@
 F 2 "Package_SO:SOIC-8_3.9x4.9mm_P1.27mm" H 1450 4900 50  0001 C CNN
 F 3 "http://www.ti.com/lit/ds/symlink/lm358.pdf" H 1450 4900 50  0001 C CNN
+F 4 "C18229" H 1450 4900 50  0001 C CNN "LCSC"
 	3    1450 4900
 	1    0    0    -1
@@
 F 2 "Resistor_SMD:R_0603_1608Metric_Pad0.98x0.95mm_HandSolder" V 2430 4700 50  0001 C CNN
 F 3 "~" H 2500 4700 50  0001 C CNN
+F 4 "C4177" H 2500 4700 50  0001 C CNN "LCSC"
 	1    2500 4700
 	0    -1   1    0
@@
 F 2 "Resistor_SMD:R_0603_1608Metric_Pad0.98x0.95mm_HandSolder" V 3130 4500 50  0001 C CNN
 F 3 "~" H 3200 4500 50  0001 C CNN
+F 4 "C22961" H 3200 4500 50  0001 C CNN "LCSC"
 	1    3200 4500
 	0    -1   1    0
@@
 F 2 "Resistor_SMD:R_0603_1608Metric_Pad0.98x0.95mm_HandSolder" V 2430 5100 50  0001 C CNN
 F 3 "~" H 2500 5100 50  0001 C CNN
+F 4 "C4177" H 2500 5100 50  0001 C CNN "LCSC"
 	1    2500 5100
 	0    -1   -1   0
@@
 F 2 "Resistor_SMD:R_0603_1608Metric_Pad0.98x0.95mm_HandSolder" V 3080 5500 50  0001 C CNN
 F 3 "~" H 3150 5500 50  0001 C CNN
+F 4 "C22961" H 3150 5500 50  0001 C CNN "LCSC"
 	1    3150 5500
 	0    -1   1    0
@@
 F 2 "Capacitor_SMD:C_0603_1608Metric_Pad1.08x0.95mm_HandSolder" H 7488 5850 50  0001 C CNN
 F 3 "~" H 7450 6000 50  0001 C CNN
+F 4 "C15849" H 7450 6000 50  0001 C CNN "LCSC"
 	1    7450 6000
 	1    0    0    -1
@@
 F 2 "Capacitor_SMD:C_0603_1608Metric_Pad1.08x0.95mm_HandSolder" H 7838 5850 50  0001 C CNN
 F 3 "~" H 7800 6000 50  0001 C CNN
+F 4 "C15849" H 7800 6000 50  0001 C CNN "LCSC"
 	1    7800 6000
 	1    0    0    -1
@@
 F 2 "Capacitor_SMD:C_0603_1608Metric_Pad1.08x0.95mm_HandSolder" H 8538 5850 50  0001 C CNN
 F 3 "~" H 8500 6000 50  0001 C CNN
+F 4 "C15849" H 8500 6000 50  0001 C CNN "LCSC"
 	1    8500 6000
 	1    0    0    -1
@@
 F 2 "Capacitor_SMD:C_0603_1608Metric_Pad1.08x0.95mm_HandSolder" H 8188 5850 50  0001 C CNN
 F 3 "~" H 8150 6000 50  0001 C CNN
+F 4 "C15849" H 8150 6000 50  0001 C CNN "LCSC"
 	1    8150 6000
 	1    0    0    -1
@@
 F 2 "Capacitor_SMD:C_0603_1608Metric_Pad1.08x0.95mm_HandSolder" H 8888 5850 50  0001 C CNN
 F 3 "~" H 8850 6000 50  0001 C CNN
+F 4 "C15849" H 8850 6000 50  0001 C CNN "LCSC"
 	1    8850 6000
 	1    0    0    -1
@@
 F 2 "Capacitor_SMD:C_0603_1608Metric_Pad1.08x0.95mm_HandSolder" H 9238 5850 50  0001 C CNN
 F 3 "~" H 9200 6000 50  0001 C CNN
+F 4 "C15849" H 9200 6000 50  0001 C CNN "LCSC"
 	1    9200 6000
 	1    0    0    -1
@@
 F 2 "Capacitor_SMD:C_0603_1608Metric_Pad1.08x0.95mm_HandSolder" H 9588 5850 50  0001 C CNN
 F 3 "~" H 9550 6000 50  0001 C CNN
+F 4 "C15849" H 9550 6000 50  0001 C CNN "LCSC"
 	1    9550 6000
 	1    0    0    -1
@@
 F 2 "Capacitor_SMD:C_0603_1608Metric_Pad1.08x0.95mm_HandSolder" H 9938 5850 50  0001 C CNN
 F 3 "~" H 9900 6000 50  0001 C CNN
+F 4 "C15849" H 9900 6000 50  0001 C CNN "LCSC"
 	1    9900 6000
 	1    0    0    -1
@@
 F 2 "Capacitor_SMD:C_0603_1608Metric_Pad1.08x0.95mm_HandSolder" H 10288 5850 50  0001 C CNN
 F 3 "~" H 10250 6000 50  0001 C CNN
+F 4 "C15849" H 10250 6000 50  0001 C CNN "LCSC"
 	1    10250 6000
 	1    0    0    -1
@@
 F 2 "Capacitor_SMD:C_0603_1608Metric_Pad1.08x0.95mm_HandSolder" H 10638 5850 50  0001 C CNN
 F 3 "~" H 10600 6000 50  0001 C CNN
+F 4 "C15849" H 10600 6000 50  0001 C CNN "LCSC"
 	1    10600 6000
 	1    0    0    -1
@@
 F 2 "Capacitor_SMD:C_0603_1608Metric_Pad1.08x0.95mm_HandSolder" H 1038 4750 50  0001 C CNN
 F 3 "~" H 1000 4900 50  0001 C CNN
+F 4 "C14663" H 1000 4900 50  0001 C CNN "LCSC"
 	1    1000 4900
 	-1   0    0    1
@@
 F 2 "Resistor_SMD:R_0603_1608Metric_Pad0.98x0.95mm_HandSolder" V 3730 5000 50  0001 C CNN
 F 3 "~" H 3800 5000 50  0001 C CNN
+F 4 "C21190" H 3800 5000 50  0001 C CNN "LCSC"
 	1    3800 5000
 	0    1    1    0
@@
 F 2 "Capacitor_SMD:C_0603_1608Metric_Pad1.08x0.95mm_HandSolder" H 4038 5100 50  0001 C CNN
 F 3 "~" H 4000 5250 50  0001 C CNN
+F 4 "C57112" H 4000 5250 50  0001 C CNN "LCSC"
 	1    4000 5250
 	1    0    0    -1
@@
 F 2 "Resistor_SMD:R_0603_1608Metric_Pad0.98x0.95mm_HandSolder" V 2030 6800 50  0001 C CNN
 F 3 "~" H 2100 6800 50  0001 C CNN
+F 4 "C21190" H 2100 6800 50  0001 C CNN "LCSC"
 	1    2100 6800
 	0    1    1    0
@@
 F 2 "Capacitor_SMD:C_0603_1608Metric_Pad1.08x0.95mm_HandSolder" H 2338 6900 50  0001 C CNN
 F 3 "~" H 2300 7050 50  0001 C CNN
+F 4 "C57112" H 2300 7050 50  0001 C CNN "LCSC"
 	1    2300 7050
 	1    0    0    -1
@@
 F 2 "Diode_SMD:D_SOD-123F" H 9900 5250 50  0001 C CNN
 F 3 "~" H 9900 5250 50  0001 C CNN
+F 4 "C64898" H 9900 5250 50  0001 C CNN "LCSC"
 	1    9900 5250
 	1    0    0    -1
@@
 F 2 "Diode_SMD:D_SOD-123F" H 9900 4800 50  0001 C CNN
 F 3 "~" H 9900 4800 50  0001 C CNN
+F 4 "C64898" H 9900 4800 50  0001 C CNN "LCSC"
 	1    9900 4800
 	1    0    0    -1
@@
 F 2 "Resistor_SMD:R_0603_1608Metric_Pad0.98x0.95mm_HandSolder" H 4400 5000 50  0001 C CNN
 F 3 "~" H 4400 5000 50  0001 C CNN
+F 4 "C21189" H 4400 5000 50  0001 C CNN "LCSC"
 	1    4400 5000
 	1    0    0    -1
@@
 F 2 "Resistor_SMD:R_0603_1608Metric_Pad0.98x0.95mm_HandSolder" H 2700 6800 50  0001 C CNN
 F 3 "~" H 2700 6800 50  0001 C CNN
+F 4 "C21189" H 2700 6800 50  0001 C CNN "LCSC"
 	1    2700 6800
 	1    0    0    -1
@@
 F 2 "" H 3200 5000 50  0001 C CNN
 F 3 "http://www.ti.com/lit/ds/symlink/lm358.pdf" H 3200 5000 50  0001 C CNN
+F 4 "C18229" H 3200 5000 50  0001 C CNN "LCSC"
 	1    3200 5000
 	1    0    0    -1
@@
 F 2 "Resistor_SMD:R_0603_1608Metric_Pad0.98x0.95mm_HandSolder" V 10430 4800 50  0001 C CNN
 F 3 "~" H 10500 4800 50  0001 C CNN
+F 4 "C21190" H 10500 4800 50  0001 C CNN "LCSC"
 	1    10500 4800
 	0    1    1    0
@@
 F 2 "Resistor_SMD:R_0603_1608Metric_Pad0.98x0.95mm_HandSolder" V 7230 4450 50  0001 C CNN
 F 3 "~" H 7300 4450 50  0001 C CNN
+F 4 "C25804" H 7300 4450 50  0001 C CNN "LCSC"
 	1    7300 4450
 	0    1    1    0
@@
 F 2 "Resistor_SMD:R_0603_1608Metric_Pad0.98x0.95mm_HandSolder" V 7230 4900 50  0001 C CNN
 F 3 "~" H 7300 4900 50  0001 C CNN
+F 4 "C25804" H 7300 4900 50  0001 C CNN "LCSC"
 	1    7300 4900
 	0    1    1    0
@@
 F 2 "Resistor_SMD:R_0603_1608Metric_Pad0.98x0.95mm_HandSolder" H 8050 4900 50  0001 C CNN
 F 3 "~" H 8050 4900 50  0001 C CNN
+F 4 "C21189" H 8050 4900 50  0001 C CNN "LCSC"
 	1    8050 4900
 	1    0    0    -1
