File: BottleBlink.kicad_sch (KiCad schematic)
At the start: 72 parts, among them J1 Arduino_Nano_v2.x, SW1 SW_DPST_x2, SW2 SW_DPST_x2, SW3 SW_DPST_x2, SW4 SW_DPST_x2, SW5 SW_DPST_x2, SW6 SW_DPST_x2

Commit message: Final fixes before production
Connections:
- net +3V3: no longer names the net of J1.17 (3V3)
Other:
- moved on the sheet: C1, C10, C11, C12, C13, C14, C15, C16, C17, C18, C19, C2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
